Commit message: enhance code

File: assets/robots/cylinder_robot.urdf (robot description, URDF)
Before this commit: robot cylinder_robot, 2 links, 1 joints
Links:
- added link camera_link
- added link imu_link
Joints:
- added joint camera_joint: type fixed, parent base_link, child camera_link, origin xyz=-0.1 0 0.5 rpy=0 0 0
- added joint imu_joint: type fixed, parent base_link, child imu_link, origin xyz=0 0 0 rpy=0 0 0
